File: analog_sensor_single_channel_R1.sch (EAGLE design)
At the start: 21 parts, among them Q1 ZVN3310A, T1 2N3904, U1 LMC6064, U2 LMC6064

Commit message: Add files via upload
Other:
- note added: "0-5V ANALOG OUT"
- note added: "ON/OFF OUTPUT"
Changed lines of the file:
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@@
 <text x="312.42" y="15.24" size="1.778" layer="91">ON/OFF COMPARATOR &amp; LED</text>
 <text x="246.38" y="-78.74" size="1.778" layer="91">UNUSED OP-AMPS (WOULD BE USED IN SUBSEQUENT CHANNEL CIRCUIT)</text>
+<text x="256.54" y="27.94" size="1.778" layer="91">0-5V ANALOG OUT</text>
+<text x="320.04" y="30.48" size="1.778" layer="91">ON/OFF OUTPUT</text>
 </plain>
 <instances>

Commit message: Add files via upload
Other:
- note added: "VOLTAGE FOLLOWER"
Changed lines of the file:
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@@
 <text x="256.54" y="27.94" size="1.778" layer="91">0-5V ANALOG OUT</text>
 <text x="320.04" y="30.48" size="1.778" layer="91">ON/OFF OUTPUT</text>
+<text x="48.26" y="86.36" size="1.778" layer="91">VOLTAGE FOLLOWER</text>
 </plain>
 <instances>
